Commit message: computer_backup_0716

File: src/localization/urdf/robot.urdf.xacro (robot description, xacro)
@@ -59,3 +59,9 @@
     <origin xyz="0 0 0" rpy="0 0 0" />
   </joint>
+<link name="lidar_link"></link>
+  <joint name="base_link" type="fixed">
+    <parent link="lidar_link" />
+    <child link="base_link" />
+    <origin xyz="-0.375 0 0" rpy="0 0 0" />
+  </joint>
 </robot>

Commit message: 1008_backup

File: src/localization/urdf/robot.urdf.xacro (robot description, xacro)
@@ -34,5 +34,5 @@
   </joint>
 </robot> -->
-<link name="base_link"></link>
+  <link name="base_link"></link>
   <!-- <link name="velodyne"> </link>
   <joint name="velodyne_joint" type="fixed">
@@ -45,5 +45,5 @@
     <parent link="base_link" />
     <child link="velodyne" />
-    <origin xyz="0.375 0 0" rpy="0 0 0" />
+    <origin xyz="0.38 0 0" rpy="0 0 0" />
   </joint>
   <link name="imu_link"> </link>
