Commit message: desktop_backup_1016

File: src/localization/urdf/robot.urdf_ys.xacro (robot description, xacro)
@@ -2,59 +2,9 @@
 <robot name="erp42" xmlns:xacro="http://www.ros.org/wiki/xacro">
   <xacro:property name="PI" value="3.1415926535897931" />
-  <!-- <link name="chassis_link"></link>
-  <link name="base_link"></link>
-  <joint name="base_link_joint" type="fixed">
-    <parent link="base_link"/>
-    <child link="chassis_link" />
-    <origin xyz="0 0 0" rpy="0 0 0" />
-  </joint>
-  <link name="velodyne"> </link>
-  <joint name="velodyne_joint" type="fixed">
-    <parent link="chassis_link" />
-    <child link="velodyne" />
-    <origin xyz="1.1 0 0.55" rpy="0 0 0" />
-  </joint>
-  <link name="imu_link"> </link>
-  <joint name="imu_joint" type="fixed">
-    <parent link="chassis_link" />
-    <child link="imu_link" />
-    <origin xyz="0 0 0" rpy="0 0 0" />
-  </joint>
-  <link name="navsat_link"> </link>
-  <joint name="navsat_joint" type="fixed">
-    <parent link="chassis_link" />
-    <child link="navsat_link" />
-    <origin xyz="0 0 0" rpy="0 0 0" />
-  </joint>
-  <link name="gps"> </link>
-  <joint name="gps_joint" type="fixed">
-    <parent link="chassis_link" />
-    <child link="gps" />
-    <origin xyz="0 0 0" rpy="0 0 0" />
-  </joint>
-</robot> -->
-<link name="base_link"></link>
-  <!-- <link name="velodyne"> </link>
-  <joint name="velodyne_joint" type="fixed">
-    <parent link="base_link" />
-    <child link="velodyne" />
-    <origin xyz="1.1 0 0.55" rpy="0 0 0" />
-  </joint> -->
-  <link name="velodyne"> </link>
-  <joint name="velodyne_joint" type="fixed">
-    <parent link="base_link" />
-    <child link="velodyne" />
-    <origin xyz="0 0 0" rpy="0 0 0" />
-  </joint>
-  <link name="imu_link"> </link>
-  <joint name="imu_joint" type="fixed">
-    <parent link="base_link" />
-    <child link="imu_link" />
-    <origin xyz="0 0 0" rpy="0 0 0" />
-  </joint>
-  <link name="gps"> </link>
-  <joint name="gps_joint" type="fixed">
-    <parent link="base_link" />
-    <child link="gps" />
+<link name="base_link_ys"></link>
+  <link name="velodyne_ys"> </link>
+  <joint name="velodyne_ys_joint" type="fixed">
+    <parent link="base_link_ys" />
+    <child link="velodyne_ys" />
     <origin xyz="0 0 0" rpy="0 0 0" />
   </joint>

Commit message: 1026 backup

File: src/localization/urdf/robot.urdf_ys.xacro (robot description, xacro)
@@ -7,5 +7,5 @@
     <parent link="base_link_ys" />
     <child link="velodyne_ys" />
-    <origin xyz="0 0 0" rpy="0 0 0" />
+    <origin xyz="0.38 0 0" rpy="0 0 0" />
   </joint>
 </robot>
